File: untitled.brd (EAGLE design)
At the start: 59.7 x 60.6 mm, 24 parts, among them IC1 ATMEGA328-20P, IC2 7805T

Commit message: Add files via upload
Connections:
- removed net N$11: 10K.1, 10KOHM.A, 330.2, C5.+, DIS1.2, IC1.20, IC1.21, IC1.7, POWER.1
- net N$6: now also 10K.1, 10KOHM.A, 330.2, C5.+, DIS1.2, IC1.20, IC1.21, IC1.7, POWER.1
Routing:
- net N$6: track 12.6 -> 186.8 mm
- net N$11: track 155.9 -> 0.00 mm
Changed lines of the file:
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@@
 <wire x1="41.91" y1="51.0794" x2="42.4688" y2="50.5206" width="0.4064" layer="16"/>
 <wire x1="42.4688" y1="50.5206" x2="48.9712" y2="50.5206" width="0.4064" layer="16"/>
-</signal>
-<signal name="N$8">
-<contactref element="33" pad="2"/>
-<contactref element="Q1" pad="2"/>
-<contactref element="IC1" pad="9"/>
-<wire x1="38.1" y1="73.66" x2="41.91" y2="73.66" width="0.4064" layer="16"/>
-<wire x1="41.91" y1="73.66" x2="43.18" y2="72.39" width="0.4064" layer="16"/>
-<wire x1="43.18" y1="72.39" x2="43.18" y2="71.12" width="0.4064" layer="16"/>
-<wire x1="43.18" y1="71.12" x2="48.26" y2="71.12" width="0.4064" layer="16"/>
-</signal>
-<signal name="N$9">
-<contactref element="33PF" pad="1"/>
-<contactref element="Q1" pad="1"/>
-<contactref element="IC1" pad="10"/>
-<wire x1="38.1" y1="76.2" x2="43.18" y2="76.2" width="0.4064" layer="16"/>
-<wire x1="43.18" y1="76.2" x2="46.99" y2="76.2" width="0.4064" layer="16"/>
-<wire x1="46.99" y1="76.2" x2="48.26" y2="74.93" width="0.4064" layer="16"/>
-</signal>
-<signal name="N$11">
 <contactref element="C5" pad="+"/>
 <contactref element="IC1" pad="7"/>
@@
 <wire x1="38.1" y1="68.58" x2="34.29" y2="68.58" width="0.4064" layer="16"/>
 <wire x1="34.29" y1="68.58" x2="33.02" y2="67.31" width="0.4064" layer="16"/>
-<wire x1="33.02" y1="67.31" x2="33.02" y2="45.72" width="0.4064" layer="16"/>
+<wire x1="33.02" y1="67.31" x2="33.02" y2="49.53" width="0.4064" layer="16"/>
+<wire x1="33.02" y1="49.53" x2="33.02" y2="45.72" width="0.4064" layer="16"/>
 <wire x1="33.02" y1="45.72" x2="34.29" y2="44.45" width="0.4064" layer="16"/>
+<wire x1="48.9712" y1="50.5206" x2="48.9712" y2="48.9712" width="0.4064" layer="16"/>
+<wire x1="48.9712" y1="48.9712" x2="48.26" y2="48.26" width="0.4064" layer="16"/>
+<wire x1="48.26" y1="48.26" x2="38.1" y2="48.26" width="0.4064" layer="16"/>
+<wire x1="38.1" y1="48.26" x2="36.83" y2="49.53" width="0.4064" layer="16"/>
+<wire x1="36.83" y1="49.53" x2="33.02" y2="49.53" width="0.4064" layer="16"/>
+</signal>
+<signal name="N$8">
+<contactref element="33" pad="2"/>
+<contactref element="Q1" pad="2"/>
+<contactref element="IC1" pad="9"/>
+<wire x1="38.1" y1="73.66" x2="41.91" y2="73.66" width="0.4064" layer="16"/>
+<wire x1="41.91" y1="73.66" x2="43.18" y2="72.39" width="0.4064" layer="16"/>
+<wire x1="43.18" y1="72.39" x2="43.18" y2="71.12" width="0.4064" layer="16"/>
+<wire x1="43.18" y1="71.12" x2="48.26" y2="71.12" width="0.4064" layer="16"/>
+</signal>
+<signal name="N$9">
+<contactref element="33PF" pad="1"/>
+<contactref element="Q1" pad="1"/>
+<contactref element="IC1" pad="10"/>
+<wire x1="38.1" y1="76.2" x2="43.18" y2="76.2" width="0.4064" layer="16"/>
+<wire x1="43.18" y1="76.2" x2="46.99" y2="76.2" width="0.4064" layer="16"/>
+<wire x1="46.99" y1="76.2" x2="48.26" y2="74.93" width="0.4064" layer="16"/>
 </signal>
 <signal name="N$13">
